Commit message: fix: Fix dg4f_gz xacro include path and add missing base_link

File: dg4f_gz/urdf/dg4f_gz.xacro (robot description, xacro)
@@ -1,10 +1,16 @@
 <?xml version="1.0"?>
 <robot name="delto_4f" xmlns:xacro="http://www.ros.org/wiki/xacro">
-    <xacro:include filename="$(find dg4f_description)/urdf/dg4f.xacro" />
+    <xacro:include filename="$(find dg4f_description)/urdf/dg4f.urdf" />
     <link name="world" />
+    <link name="base_link" />
     <joint name="world_to_base_fixed" type="fixed">
         <parent link="world" />
         <child link="base_link" />
         <origin xyz="0 0 0.1" rpy="0 0 0" />
+    </joint>
+    <joint name="base_joint" type="fixed">
+        <parent link="base_link" />
+        <child link="l_dg_mount" />
+        <origin xyz="0 0 0" rpy="0 0 0" />
     </joint>
     <ros2_control name="GazeboSimSystem" type="system">
